Commit message: added joystick control

File: description/robot_core.xacro (robot description, xacro)
@@ -50,5 +50,5 @@
          <collision>
             <geometry>
-                <cylinder length="0.04" radius="0.05" />
+                <sphere radius="0.05" />
             </geometry>
         </collision>
@@ -76,5 +76,5 @@
         <collision>
             <geometry>
-                <cylinder length="0.04" radius="0.05" />
+                <sphere radius="0.05" />
             </geometry>
         </collision>

File: description/ros2_control.xacro (robot description, xacro)
@@ -8,5 +8,5 @@
             <command_interface name='velocity'>
                 <param name='min'>-10</param>
-                <param name='max'>10</param>
+                <param name='max'>50</param>
             </command_interface>
             <state_interface name='velocity'/>
@@ -16,5 +16,5 @@
             <command_interface name='velocity'>
                 <param name='min'>-10</param>
-                <param name='max'>10</param>
+                <param name='max'>50</param>
             </command_interface>
             <state_interface name='velocity'/>
